File: bootarooni.sch (KiCad schematic (older format))
At the start: 25 parts, among them J1 USB_B_Micro, U1 74LS07, U2 Pico_USB, U3 ADUM3160, U4 74LCX541, U5 74AHCT1G125, U6 74LS299, U7 74LS299, U8 74LS299

Commit message: adding footprints and zeroing in on component values
Parts:
- C1, C2, C3, C4, C5, C6, C7, C8, C9: footprint (none) -> Capacitor_SMD:C_0805_2012Metric
- R3, R4: value R -> 27K
Changed lines of the file:
@@
 F 0 "C4" H 2415 1346 50  0000 L CNN
 F 1 "0.1uF" H 2415 1255 50  0000 L CNN
-F 2 "" H 2338 1150 50  0001 C CNN
+F 2 "Capacitor_SMD:C_0805_2012Metric" H 2338 1150 50  0001 C CNN
 F 3 "~" H 2300 1300 50  0001 C CNN
 	1    2300 1300
@@
 F 0 "C6" H 2665 2096 50  0000 L CNN
 F 1 "0.1uF" H 2665 2005 50  0000 L CNN
-F 2 "" H 2588 1900 50  0001 C CNN
+F 2 "Capacitor_SMD:C_0805_2012Metric" H 2588 1900 50  0001 C CNN
 F 3 "~" H 2550 2050 50  0001 C CNN
 	1    2550 2050
@@
 F 0 "C9" H 4415 1346 50  0000 L CNN
 F 1 "0.1uF" H 4415 1255 50  0000 L CNN
-F 2 "" H 4338 1150 50  0001 C CNN
+F 2 "Capacitor_SMD:C_0805_2012Metric" H 4338 1150 50  0001 C CNN
 F 3 "~" H 4300 1300 50  0001 C CNN
 	1    4300 1300
@@
 F 0 "C8" H 4165 2146 50  0000 L CNN
 F 1 "0.1uF" H 4165 2055 50  0000 L CNN
-F 2 "" H 4088 1950 50  0001 C CNN
+F 2 "Capacitor_SMD:C_0805_2012Metric" H 4088 1950 50  0001 C CNN
 F 3 "~" H 4050 2100 50  0001 C CNN
 	1    4050 2100
@@
 P 5300 4250
 F 0 "R3" H 5370 4296 50  0000 L CNN
-F 1 "R" H 5370 4205 50  0000 L CNN
+F 1 "27K" H 5370 4205 50  0000 L CNN
 F 2 "" V 5230 4250 50  0001 C CNN
 F 3 "~" H 5300 4250 50  0001 C CNN
@@
 P 5450 6300
 F 0 "R4" H 5520 6346 50  0000 L CNN
-F 1 "R" H 5520 6255 50  0000 L CNN
+F 1 "27K" H 5520 6255 50  0000 L CNN
 F 2 "" V 5380 6300 50  0001 C CNN
 F 3 "~" H 5450 6300 50  0001 C CNN
@@
 F 0 "C2" H 1650 6600 50  0000 R CNN
 F 1 "0.1uF" H 1650 6800 50  0000 R CNN
-F 2 "" H 1738 6550 50  0001 C CNN
+F 2 "Capacitor_SMD:C_0805_2012Metric" H 1738 6550 50  0001 C CNN
 F 3 "~" H 1700 6700 50  0001 C CNN
 	1    1700 6700
@@
 F 0 "C3" H 2000 6600 50  0000 R CNN
 F 1 "0.1uF" H 2000 6800 50  0000 R CNN
-F 2 "" H 2088 6550 50  0001 C CNN
+F 2 "Capacitor_SMD:C_0805_2012Metric" H 2088 6550 50  0001 C CNN
 F 3 "~" H 2050 6700 50  0001 C CNN
 	1    2050 6700
@@
 F 0 "C5" H 2350 6600 50  0000 R CNN
 F 1 "0.1uF" H 2350 6800 50  0000 R CNN
-F 2 "" H 2438 6550 50  0001 C CNN
+F 2 "Capacitor_SMD:C_0805_2012Metric" H 2438 6550 50  0001 C CNN
 F 3 "~" H 2400 6700 50  0001 C CNN
 	1    2400 6700
@@
 F 0 "C7" H 2700 6600 50  0000 R CNN
 F 1 "0.1uF" H 2700 6800 50  0000 R CNN
-F 2 "" H 2788 6550 50  0001 C CNN
+F 2 "Capacitor_SMD:C_0805_2012Metric" H 2788 6550 50  0001 C CNN
 F 3 "~" H 2750 6700 50  0001 C CNN
 	1    2750 6700
@@
 F 0 "C1" H 1300 6600 50  0000 R CNN
 F 1 "0.1uF" H 1300 6800 50  0000 R CNN
-F 2 "" H 1388 6550 50  0001 C CNN
+F 2 "Capacitor_SMD:C_0805_2012Metric" H 1388 6550 50  0001 C CNN
 F 3 "~" H 1350 6700 50  0001 C CNN
 	1    1350 6700

Commit message: fixing up voltage dividers for pull-up footprints for most parts
Parts:
- removed RN1: R_Network04, Resistor_THT:R_Array_SIP5, symbol Device:R_Network04
- added RN1, RN2: R_Pack04, symbol Device:R_Pack04
- J1: footprint (none) -> Connector_USB:USB_Micro-B_Amphenol_10103594-0001LF_Horizontal
- R1, R2, R3, R4: footprint (none) -> Resistor_SMD:R_0805_2012Metric
- TP1: footprint (none) -> TestPoint:TestPoint_Pad_D2.0mm
Connections:
- wire segments 174 -> 193
Changed lines of the file:
@@
 F 0 "R1" V 1900 1500 50  0000 C CNN
 F 1 "24R" V 1900 1650 50  0000 C CNN
-F 2 "" V 1930 1550 50  0001 C CNN
+F 2 "Resistor_SMD:R_0805_2012Metric" V 1930 1550 50  0001 C CNN
 F 3 "~" H 2000 1550 50  0001 C CNN
 	1    2000 1550
@@
 F 0 "R2" V 1900 1750 50  0000 C CNN
 F 1 "24R" V 1900 1600 50  0000 C CNN
-F 2 "" V 1930 1650 50  0001 C CNN
+F 2 "Resistor_SMD:R_0805_2012Metric" V 1930 1650 50  0001 C CNN
 F 3 "~" H 2000 1650 50  0001 C CNN
 	1    2000 1650
@@
 F 0 "J1" H 1407 2017 50  0000 C CNN
 F 1 "USB_B_Micro" H 1407 1926 50  0000 C CNN
-F 2 "" H 1500 1500 50  0001 C CNN
+F 2 "Connector_USB:USB_Micro-B_Amphenol_10103594-0001LF_Horizontal" H 1500 1500 50  0001 C CNN
 F 3 "~" H 1500 1500 50  0001 C CNN
 	1    1350 1550
@@
 F 0 "R3" H 5370 4296 50  0000 L CNN
 F 1 "27K" H 5370 4205 50  0000 L CNN
-F 2 "" V 5230 4250 50  0001 C CNN
+F 2 "Resistor_SMD:R_0805_2012Metric" V 5230 4250 50  0001 C CNN
 F 3 "~" H 5300 4250 50  0001 C CNN
 	1    5300 4250
@@
 F 0 "R4" H 5520 6346 50  0000 L CNN
 F 1 "27K" H 5520 6255 50  0000 L CNN
-F 2 "" V 5380 6300 50  0001 C CNN
+F 2 "Resistor_SMD:R_0805_2012Metric" V 5380 6300 50  0001 C CNN
 F 3 "~" H 5450 6300 50  0001 C CNN
 	1    5450 6300
@@
 F 0 "TP1" V 8895 2022 50  0000 C CNN
 F 1 "TestPoint" V 8804 2022 50  0000 C CNN
-F 2 "" H 8900 1950 50  0001 C CNN
+F 2 "TestPoint:TestPoint_Pad_D2.0mm" H 8900 1950 50  0001 C CNN
 F 3 "~" H 8900 1950 50  0001 C CNN
 	1    8700 1950
@@
 	10650 1450 10650 1350
 $Comp
-L Device:R_Network04 RN1
-U 1 1 604C8EB1
-P 7650 3450
-F 0 "RN1" H 7838 3496 50  0000 L CNN
-F 1 "R_Network04" H 7838 3405 50  0000 L CNN
-F 2 "Resistor_THT:R_Array_SIP5" V 7925 3450 50  0001 C CNN
-F 3 "http://www.vishay.com/docs/31509/csc.pdf" H 7650 3450 50  0001 C CNN
-	1    7650 3450
-	1    0    0    -1
-$EndComp
-$Comp
 L power:+5V #PWR01
 U 1 1 604CC8F0
@@
 $EndComp
 Wire Wire Line
-	7450 3150 7450 3250
+	7450 3150 7450 3200
 Wire Wire Line
 	7800 3900 7450 3900
@@
 Connection ~ 7450 3900
 Wire Wire Line
-	7450 3900 7350 3900
-Wire Wire Line
 	7550 3650 7550 4250
 Connection ~ 7550 4250
 Wire Wire Line
-	7550 4250 7350 4250
-Wire Wire Line
 	7650 3650 7650 4600
 Connection ~ 7650 4600
 Wire Wire Line
-	7650 4600 7350 4600
-Wire Wire Line
 	7750 3650 7750 4950
 Connection ~ 7750 4950
-Wire Wire Line
-	7750 4950 7350 4950
 $Comp
 L Device:C C2
@@
 Wire Wire Line
 	1350 7400 850  7400
+Wire Wire Line
+	7450 3900 7350 3900
+Wire Wire Line
+	7550 4250 7350 4250
+Wire Wire Line
+	7650 4600 7350 4600
+Wire Wire Line
+	7750 4950 7350 4950
+$Comp
+L power:GND #PWR02
+U 1 1 603F76C6
+P 7750 5750
+F 0 "#PWR02" H 7750 5500 50  0001 C CNN
+F 1 "GND" H 7755 5577 50  0000 C CNN
+F 2 "" H 7750 5750 50  0001 C CNN
+F 3 "" H 7750 5750 50  0001 C CNN
+	1    7750 5750
+	1    0    0    -1
+$EndComp
+Wire Wire Line
+	7750 5750 7750 5600
+Wire Wire Line
+	7750 5150 7750 4950
+Wire Wire Line
+	7650 5150 7650 4600
+Wire Wire Line
+	7550 4250 7550 5150
+Wire Wire Line
+	7450 5150 7450 3900
+$Comp
+L Device:R_Pack04 RN1
+U 1 1 6042F432
+P 7650 3450
+F 0 "RN1" H 7838 3496 50  0000 L CNN
+F 1 "R_Pack04" H 7838 3405 50  0000 L CNN
+F 2 "" V 7925 3450 50  0001 C CNN
+F 3 "~" H 7650 3450 50  0001 C CNN
+	1    7650 3450
+	1    0    0    -1
+$EndComp
+$Comp
+L Device:R_Pack04 RN2
+U 1 1 604348FC
+P 7650 5350
+F 0 "RN2" H 7838 5396 50  0000 L CNN
+F 1 "R_Pack04" H 7838 5305 50  0000 L CNN
+F 2 "" V 7925 5350 50  0001 C CNN
+F 3 "~" H 7650 5350 50  0001 C CNN
+	1    7650 5350
+	1    0    0    -1
+$EndComp
+Wire Wire Line
+	7650 5550 7650 5600
+Wire Wire Line
+	7650 5600 7750 5600
+Connection ~ 7750 5600
+Wire Wire Line
+	7750 5600 7750 5550
+Wire Wire Line
+	7650 5600 7550 5600
+Wire Wire Line
+	7450 5600 7450 5550
+Connection ~ 7650 5600
+Wire Wire Line
+	7550 5600 7550 5550
+Connection ~ 7550 5600
+Wire Wire Line
+	7550 5600 7450 5600
+Wire Wire Line
+	7450 3200 7550 3200
+Wire Wire Line
+	7750 3200 7750 3250
+Connection ~ 7450 3200
+Wire Wire Line
+	7450 3200 7450 3250
+Wire Wire Line
+	7550 3200 7550 3250
+Connection ~ 7550 3200
+Wire Wire Line
+	7550 3200 7650 3200
+Wire Wire Line
+	7650 3200 7650 3250
+Connection ~ 7650 3200
+Wire Wire Line
+	7650 3200 7750 3200
 $EndSCHEMATC

Commit message: Adding some NCs on schematic Rough layout on board
Parts:
- removed RN1: R_Pack04, symbol Device:R_Pack04
- removed U1: 74LS07, Package_SO:SOIC-14_3.9x8.7mm_P1.27mm, symbol 74xx:74LS07
- added U1: 74LS05, Package_SO:SOIC-14_3.9x8.7mm_P1.27mm, symbol 74xx:74LS05
- RN1: renamed from RN2; value R_Pack04 -> 47K; footprint (none) -> bootarooni:SOIC-8
Connections:
- net labels added: EXT_GND, EXT_V, P_R_~W~, P_~DEVSEL~, P_~IOSEL~, P_~STROBE~, P_ϕ1
- wire segments 193 -> 181
- no-connect marks 14 -> 17
Changed lines of the file:
@@
 These test points connect to the\ncorresponding test points on \nthe Pi Pico itself.
-$Comp
-L 74xx:74LS07 U1
-U 7 1 6030A1A1
-P 850 6900
-F 0 "U1" H 950 7250 50  0000 L CNN
-F 1 "74LS07" V 1100 6600 50  0000 L CNN
-F 2 "Package_SO:SOIC-14_3.9x8.7mm_P1.27mm" H 850 6900 50  0001 C CNN
-F 3 "www.ti.com/lit/ds/symlink/sn74ls07.pdf" H 850 6900 50  0001 C CNN
-	7    850  6900
-	1    0    0    -1
-$EndComp
 $Comp
 L power:GND #PWR0105
@@
 Text Label 9050 4150 2    50   ~ 0
 D7
-$Comp
-L 74xx:74LS07 U1
-U 1 1 60421AF4
-P 8100 3900
-F 0 "U1" H 8300 3850 50  0000 C CNN
-F 1 "74LS07" H 8300 3750 50  0000 C CNN
-F 2 "Package_SO:SOIC-14_3.9x8.7mm_P1.27mm" H 8100 3900 50  0001 C CNN
-F 3 "www.ti.com/lit/ds/symlink/sn74ls07.pdf" H 8100 3900 50  0001 C CNN
-	1    8100 3900
-	1    0    0    -1
-$EndComp
-$Comp
-L 74xx:74LS07 U1
-U 3 1 60423273
-P 8100 4600
-F 0 "U1" H 8300 4550 50  0000 C CNN
-F 1 "74LS07" H 8300 4450 50  0000 C CNN
-F 2 "Package_SO:SOIC-14_3.9x8.7mm_P1.27mm" H 8100 4600 50  0001 C CNN
-F 3 "www.ti.com/lit/ds/symlink/sn74ls07.pdf" H 8100 4600 50  0001 C CNN
-	3    8100 4600
-	1    0    0    -1
-$EndComp
-$Comp
-L 74xx:74LS07 U1
-U 2 1 60434CFD
-P 8100 4250
-F 0 "U1" H 8300 4200 50  0000 C CNN
-F 1 "74LS07" H 8300 4100 50  0000 C CNN
-F 2 "Package_SO:SOIC-14_3.9x8.7mm_P1.27mm" H 8100 4250 50  0001 C CNN
-F 3 "www.ti.com/lit/ds/symlink/sn74ls07.pdf" H 8100 4250 50  0001 C CNN
-	2    8100 4250
-	1    0    0    -1
-$EndComp
-$Comp
-L 74xx:74LS07 U1
-U 4 1 60435ED0
-P 8100 4950
-F 0 "U1" H 8300 4900 50  0000 C CNN
-F 1 "74LS07" H 8300 4800 50  0000 C CNN
-F 2 "Package_SO:SOIC-14_3.9x8.7mm_P1.27mm" H 8100 4950 50  0001 C CNN
-F 3 "www.ti.com/lit/ds/symlink/sn74ls07.pdf" H 8100 4950 50  0001 C CNN
-	4    8100 4950
-	1    0    0    -1
-$EndComp
 Text Label 8400 3900 0    50   ~ 0
 ~NMI~
@@
 Wire Wire Line
 	10650 1450 10650 1350
-$Comp
-L power:+5V #PWR01
-U 1 1 604CC8F0
-P 7450 3150
-F 0 "#PWR01" H 7450 3000 50  0001 C CNN
-F 1 "+5V" H 7465 3323 50  0000 C CNN
-F 2 "" H 7450 3150 50  0001 C CNN
-F 3 "" H 7450 3150 50  0001 C CNN
-	1    7450 3150
-	1    0    0    -1
-$EndComp
-Wire Wire Line
-	7450 3150 7450 3200
 Wire Wire Line
 	7800 3900 7450 3900
@@
 Wire Wire Line
 	7800 4950 7750 4950
-Wire Wire Line
-	7450 3650 7450 3900
 Connection ~ 7450 3900
-Wire Wire Line
-	7550 3650 7550 4250
 Connection ~ 7550 4250
-Wire Wire Line
-	7650 3650 7650 4600
 Connection ~ 7650 4600
-Wire Wire Line
-	7750 3650 7750 4950
 Connection ~ 7750 4950
 $Comp
@@
 Wire Wire Line
 	2750 6400 2750 6550
-Connection ~ 850  6400
 Wire Wire Line
 	2750 6850 2750 7400
 Wire Wire Line
 	2750 7400 2400 7400
-Connection ~ 850  7400
 Wire Wire Line
 	1700 6550 1700 6400
@@
 Wire Wire Line
 	7450 5150 7450 3900
+Wire Wire Line
+	7650 5550 7650 5600
+Wire Wire Line
+	7650 5600 7750 5600
+Connection ~ 7750 5600
+Wire Wire Line
+	7750 5600 7750 5550
+Wire Wire Line
+	7650 5600 7550 5600
+Wire Wire Line
+	7450 5600 7450 5550
+Connection ~ 7650 5600
+Wire Wire Line
+	7550 5600 7550 5550
+Connection ~ 7550 5600
+Wire Wire Line
+	7550 5600 7450 5600
+$Comp
+L 74xx:74LS05 U1
+U 7 1 6048CAD2
+P 850 6900
+F 0 "U1" H 1080 6946 50  0000 L CNN
+F 1 "74LS05" H 1080 6855 50  0000 L CNN
+F 2 "Package_SO:SOIC-14_3.9x8.7mm_P1.27mm" H 850 6900 50  0001 C CNN
+F 3 "http://www.ti.com/lit/gpn/sn74LS05" H 850 6900 50  0001 C CNN
+	7    850  6900
+	1    0    0    -1
+$EndComp
+Connection ~ 850  6400
+Connection ~ 850  7400
+$Comp
+L 74xx:74LS05 U1
+U 1 1 6048E273
+P 8100 3900
+F 0 "U1" H 8100 4217 50  0000 C CNN
+F 1 "74LS05" H 8100 4126 50  0000 C CNN
+F 2 "Package_SO:SOIC-14_3.9x8.7mm_P1.27mm" H 8100 3900 50  0001 C CNN
+F 3 "http://www.ti.com/lit/gpn/sn74LS05" H 8100 3900 50  0001 C CNN
+	1    8100 3900
+	1    0    0    -1
+$EndComp
+$Comp
+L 74xx:74LS05 U1
+U 2 1 6048EF63
+P 8100 4250
+F 0 "U1" H 8100 4567 50  0000 C CNN
+F 1 "74LS05" H 8100 4476 50  0000 C CNN
+F 2 "Package_SO:SOIC-14_3.9x8.7mm_P1.27mm" H 8100 4250 50  0001 C CNN
+F 3 "http://www.ti.com/lit/gpn/sn74LS05" H 8100 4250 50  0001 C CNN
+	2    8100 4250
+	1    0    0    -1
+$EndComp
+$Comp
+L 74xx:74LS05 U1
+U 3 1 6048FD1A
+P 8100 4600
+F 0 "U1" H 8100 4917 50  0000 C CNN
+F 1 "74LS05" H 8100 4826 50  0000 C CNN
+F 2 "Package_SO:SOIC-14_3.9x8.7mm_P1.27mm" H 8100 4600 50  0001 C CNN
+F 3 "http://www.ti.com/lit/gpn/sn74LS05" H 8100 4600 50  0001 C CNN
+	3    8100 4600
+	1    0    0    -1
+$EndComp
+$Comp
+L 74xx:74LS05 U1
+U 4 1 60490D69
+P 8100 4950
+F 0 "U1" H 8100 5267 50  0000 C CNN
+F 1 "74LS05" H 8100 5176 50  0000 C CNN
+F 2 "Package_SO:SOIC-14_3.9x8.7mm_P1.27mm" H 8100 4950 50  0001 C CNN
+F 3 "http://www.ti.com/lit/gpn/sn74LS05" H 8100 4950 50  0001 C CNN
+	4    8100 4950
+	1    0    0    -1
+$EndComp
 $Comp
 L Device:R_Pack04 RN1
-U 1 1 6042F432
-P 7650 3450
-F 0 "RN1" H 7838 3496 50  0000 L CNN
-F 1 "R_Pack04" H 7838 3405 50  0000 L CNN
-F 2 "" V 7925 3450 50  0001 C CNN
-F 3 "~" H 7650 3450 50  0001 C CNN
-	1    7650 3450
-	1    0    0    -1
-$EndComp
-$Comp
-L Device:R_Pack04 RN2
 U 1 1 604348FC
 P 7650 5350
-F 0 "RN2" H 7838 5396 50  0000 L CNN
-F 1 "R_Pack04" H 7838 5305 50  0000 L CNN
-F 2 "" V 7925 5350 50  0001 C CNN
+F 0 "RN1" H 7838 5396 50  0000 L CNN
+F 1 "47K" H 7838 5305 50  0000 L CNN
+F 2 "bootarooni:SOIC-8" V 7925 5350 50  0001 C CNN
 F 3 "~" H 7650 5350 50  0001 C CNN
 	1    7650 5350
 	1    0    0    -1
 $EndComp
-Wire Wire Line
-	7650 5550 7650 5600
-Wire Wire Line
-	7650 5600 7750 5600
-Connection ~ 7750 5600
-Wire Wire Line
-	7750 5600 7750 5550
-Wire Wire Line
-	7650 5600 7550 5600
-Wire Wire Line
-	7450 5600 7450 5550
-Connection ~ 7650 5600
-Wire Wire Line
-	7550 5600 7550 5550
-Connection ~ 7550 5600
-Wire Wire Line
-	7550 5600 7450 5600
-Wire Wire Line
-	7450 3200 7550 3200
-Wire Wire Line
-	7750 3200 7750 3250
-Connection ~ 7450 3200
-Wire Wire Line
-	7450 3200 7450 3250
-Wire Wire Line
-	7550 3200 7550 3250
-Connection ~ 7550 3200
-Wire Wire Line
-	7550 3200 7650 3200
-Wire Wire Line
-	7650 3200 7650 3250
-Connection ~ 7650 3200
-Wire Wire Line
-	7650 3200 7750 3200
+Text Label 1950 1050 0    50   ~ 0
+EXT_V
+Text Label 1650 2350 0    50   ~ 0
+EXT_GND
+NoConn ~ 3800 6800
+NoConn ~ 3800 6700
+NoConn ~ 3800 6600
+Text Label 3800 6500 2    50   ~ 0
+P_~STROBE~
+Text Label 3800 6400 2    50   ~ 0
+P_R_~W~
+Text Label 3800 6300 2    50   ~ 0
+P_ϕ1
+Text Label 3800 6200 2    50   ~ 0
+P_~DEVSEL~
+Text Label 3800 6100 2    50   ~ 0
+P_~IOSEL~
 $EndSCHEMATC
