File: bootarooni.sch (KiCad schematic (older format))
At the start: 34 parts, among them J1 USB_B_Micro, U1 74LS05, U2 Pico_USB, U3 ADUM3160, U4 74LCX541, U5 74AHCT1G125, U6 74LS299, U7 74LS299, U8 74LS299

Commit message: final v1; board, digikey, and stencil orders submitted
Parts:
- C1, C2, C3, C4, C5, C6, C7, C8, C9: Digikey P/N (none) -> 399-8000-1-ND
- D1, D2, D3, D4: Digikey P/N (none) -> 160-1423-1-ND
- J1: Digikey P/N (none) -> 609-4050-1-ND
- R1, R2: Digikey P/N (none) -> P24.0CCT-ND
- R3, R4: Digikey P/N (none) -> P27.0KCCT-ND
- RN1: Digikey P/N (none) -> Y10473CT-ND
- RN2: Digikey P/N (none) -> Y7471CT-ND
- U1: Digikey P/N (none) -> 296-1630-1-ND
- U3: Digikey P/N (none) -> ADUM3160BRWZ-RLCT-ND
- U4: Digikey P/N (none) -> 74LCX541WMXCT-ND
- U5: Digikey P/N (none) -> M74VHC1GT125DF1GOSCT-ND
- U6, U7, U8: Digikey P/N (none) -> 296-4277-5-ND
Changed lines of the file:
@@
 F 2 "Resistor_SMD:R_0805_2012Metric" V 1930 1550 50  0001 C CNN
 F 3 "~" H 2000 1550 50  0001 C CNN
+F 4 "P24.0CCT-ND" H 2000 1550 50  0001 C CNN "Digikey P/N"
 	1    2000 1550
 	0    1    1    0
@@
 F 2 "Resistor_SMD:R_0805_2012Metric" V 1930 1650 50  0001 C CNN
 F 3 "~" H 2000 1650 50  0001 C CNN
+F 4 "P24.0CCT-ND" H 2000 1650 50  0001 C CNN "Digikey P/N"
 	1    2000 1650
 	0    -1   -1   0
@@
 F 2 "Connector_USB:USB_Micro-B_Amphenol_10103594-0001LF_Horizontal" H 1500 1500 50  0001 C CNN
 F 3 "~" H 1500 1500 50  0001 C CNN
+F 4 "609-4050-1-ND" H 1350 1550 50  0001 C CNN "Digikey P/N"
 	1    1350 1550
 	1    0    0    -1
@@
 F 2 "Package_SO:SOIC-16W_7.5x10.3mm_P1.27mm" H 3350 950 50  0001 C CNN
 F 3 "https://www.analog.com/media/en/technical-documentation/data-sheets/ADuM3160.pdf" H 3150 1650 50  0001 C CNN
+F 4 "ADUM3160BRWZ-RLCT-ND" H 3350 1650 50  0001 C CNN "Digikey P/N"
 	1    3350 1650
 	1    0    0    -1
@@
 F 2 "Capacitor_SMD:C_0805_2012Metric" H 2338 1150 50  0001 C CNN
 F 3 "~" H 2300 1300 50  0001 C CNN
+F 4 "399-8000-1-ND" H 2300 1300 50  0001 C CNN "Digikey P/N"
 	1    2300 1300
 	1    0    0    -1
@@
 F 2 "Capacitor_SMD:C_0805_2012Metric" H 2588 1900 50  0001 C CNN
 F 3 "~" H 2550 2050 50  0001 C CNN
+F 4 "399-8000-1-ND" H 2550 2050 50  0001 C CNN "Digikey P/N"
 	1    2550 2050
 	1    0    0    -1
@@
 F 2 "Capacitor_SMD:C_0805_2012Metric" H 4338 1150 50  0001 C CNN
 F 3 "~" H 4300 1300 50  0001 C CNN
+F 4 "399-8000-1-ND" H 4300 1300 50  0001 C CNN "Digikey P/N"
 	1    4300 1300
 	1    0    0    -1
@@
 F 2 "Capacitor_SMD:C_0805_2012Metric" H 4088 1950 50  0001 C CNN
 F 3 "~" H 4050 2100 50  0001 C CNN
+F 4 "399-8000-1-ND" H 4050 2100 50  0001 C CNN "Digikey P/N"
 	1    4050 2100
 	1    0    0    -1
@@
 F 2 "Package_SO:SOIC-20W_7.5x12.8mm_P1.27mm" H 4300 6600 50  0001 C CNN
 F 3 "http://www.ti.com/lit/gpn/sn74LS541" H 4300 6600 50  0001 C CNN
+F 4 "74LCX541WMXCT-ND" H 4300 6600 50  0001 C CNN "Digikey P/N"
 	1    4300 6600
 	-1   0    0    -1
@@
 F 2 "Package_SO:SOIC-20W_7.5x12.8mm_P1.27mm" H 6300 4000 50  0001 C CNN
 F 3 "http://www.ti.com/lit/gpn/sn74LS299" H 6300 4000 50  0001 C CNN
+F 4 "296-4277-5-ND" H 6300 4000 50  0001 C CNN "Digikey P/N"
 	1    6300 4000
 	1    0    0    -1
@@
 F 2 "Package_SO:SOIC-20W_7.5x12.8mm_P1.27mm" H 6300 5950 50  0001 C CNN
 F 3 "http://www.ti.com/lit/gpn/sn74LS299" H 6300 5950 50  0001 C CNN
+F 4 "296-4277-5-ND" H 6300 5950 50  0001 C CNN "Digikey P/N"
 	1    6300 5950
 	1    0    0    -1
@@
 F 2 "Resistor_SMD:R_0805_2012Metric" V 5230 4250 50  0001 C CNN
 F 3 "~" H 5300 4250 50  0001 C CNN
+F 4 "P27.0KCCT-ND" H 5300 4250 50  0001 C CNN "Digikey P/N"
 	1    5300 4250
 	1    0    0    -1
@@
 F 2 "Resistor_SMD:R_0805_2012Metric" V 5380 6300 50  0001 C CNN
 F 3 "~" H 5450 6300 50  0001 C CNN
+F 4 "P27.0KCCT-ND" H 5450 6300 50  0001 C CNN "Digikey P/N"
 	1    5450 6300
 	1    0    0    -1
@@
 F 2 "Package_TO_SOT_SMD:SOT-353_SC-70-5" H 4800 3900 50  0001 C CNN
 F 3 "http://www.ti.com/lit/sg/scyt129e/scyt129e.pdf" H 4800 3900 50  0001 C CNN
+F 4 "M74VHC1GT125DF1GOSCT-ND" H 4800 3900 50  0001 C CNN "Digikey P/N"
 	1    4800 3900
 	0    1    -1   0
@@
 F 2 "Package_SO:SOIC-20W_7.5x12.8mm_P1.27mm" H 6300 2050 50  0001 C CNN
 F 3 "http://www.ti.com/lit/gpn/sn74LS299" H 6300 2050 50  0001 C CNN
+F 4 "296-4277-5-ND" H 6300 2050 50  0001 C CNN "Digikey P/N"
 	1    6300 2050
 	1    0    0    -1
@@
 F 2 "Capacitor_SMD:C_0805_2012Metric" H 1738 6550 50  0001 C CNN
 F 3 "~" H 1700 6700 50  0001 C CNN
+F 4 "399-8000-1-ND" H 1700 6700 50  0001 C CNN "Digikey P/N"
 	1    1700 6700
 	-1   0    0    1
@@
 F 2 "Capacitor_SMD:C_0805_2012Metric" H 2088 6550 50  0001 C CNN
 F 3 "~" H 2050 6700 50  0001 C CNN
+F 4 "399-8000-1-ND" H 2050 6700 50  0001 C CNN "Digikey P/N"
 	1    2050 6700
 	-1   0    0    1
@@
 F 2 "Capacitor_SMD:C_0805_2012Metric" H 2788 6550 50  0001 C CNN
 F 3 "~" H 2750 6700 50  0001 C CNN
+F 4 "399-8000-1-ND" H 2750 6700 50  0001 C CNN "Digikey P/N"
 	1    2750 6700
 	-1   0    0    1
@@
 F 2 "Capacitor_SMD:C_0805_2012Metric" H 2438 6550 50  0001 C CNN
 F 3 "~" H 2400 6700 50  0001 C CNN
+F 4 "399-8000-1-ND" H 2400 6700 50  0001 C CNN "Digikey P/N"
 	1    2400 6700
 	-1   0    0    1
@@
 F 2 "Capacitor_SMD:C_0805_2012Metric" H 1388 6550 50  0001 C CNN
 F 3 "~" H 1350 6700 50  0001 C CNN
+F 4 "399-8000-1-ND" H 1350 6700 50  0001 C CNN "Digikey P/N"
 	1    1350 6700
 	-1   0    0    1
@@
 F 2 "Package_SO:SOIC-14_3.9x8.7mm_P1.27mm" H 850 6900 50  0001 C CNN
 F 3 "http://www.ti.com/lit/gpn/sn74LS05" H 850 6900 50  0001 C CNN
+F 4 "296-1630-1-ND" H 850 6900 50  0001 C CNN "Digikey P/N"
 	7    850  6900
 	1    0    0    -1
@@
 F 2 "Package_SO:SOIC-14_3.9x8.7mm_P1.27mm" H 8100 3900 50  0001 C CNN
 F 3 "http://www.ti.com/lit/gpn/sn74LS05" H 8100 3900 50  0001 C CNN
+F 4 "296-1630-1-ND" H 8100 3900 50  0001 C CNN "Digikey P/N"
 	1    8100 3900
 	1    0    0    -1
@@
 F 2 "Package_SO:SOIC-14_3.9x8.7mm_P1.27mm" H 8100 4250 50  0001 C CNN
 F 3 "http://www.ti.com/lit/gpn/sn74LS05" H 8100 4250 50  0001 C CNN
+F 4 "296-1630-1-ND" H 8100 4250 50  0001 C CNN "Digikey P/N"
 	2    8100 4250
 	1    0    0    -1
@@
 F 2 "Package_SO:SOIC-14_3.9x8.7mm_P1.27mm" H 8100 4600 50  0001 C CNN
 F 3 "http://www.ti.com/lit/gpn/sn74LS05" H 8100 4600 50  0001 C CNN
+F 4 "296-1630-1-ND" H 8100 4600 50  0001 C CNN "Digikey P/N"
 	3    8100 4600
 	1    0    0    -1
@@
 F 2 "Package_SO:SOIC-14_3.9x8.7mm_P1.27mm" H 8100 4950 50  0001 C CNN
 F 3 "http://www.ti.com/lit/gpn/sn74LS05" H 8100 4950 50  0001 C CNN
+F 4 "296-1630-1-ND" H 8100 4950 50  0001 C CNN "Digikey P/N"
 	4    8100 4950
 	1    0    0    -1
@@
 F 2 "bootarooni:SOIC-8" V 7925 5350 50  0001 C CNN
 F 3 "~" H 7650 5350 50  0001 C CNN
+F 4 "Y10473CT-ND" H 7650 5350 50  0001 C CNN "Digikey P/N"
 	1    7650 5350
 	1    0    0    -1
@@
 F 2 "Package_SO:SOIC-14_3.9x8.7mm_P1.27mm" H 8050 3050 50  0001 C CNN
 F 3 "http://www.ti.com/lit/gpn/sn74LS05" H 8050 3050 50  0001 C CNN
+F 4 "296-1630-1-ND" H 8050 3050 50  0001 C CNN "Digikey P/N"
 	5    8050 3050
 	1    0    0    -1
@@
 F 2 "Package_SO:SOIC-14_3.9x8.7mm_P1.27mm" H 8050 2550 50  0001 C CNN
 F 3 "http://www.ti.com/lit/gpn/sn74LS05" H 8050 2550 50  0001 C CNN
+F 4 "296-1630-1-ND" H 8050 2550 50  0001 C CNN "Digikey P/N"
 	6    8050 2550
 	1    0    0    -1
@@
 F 2 "bootarooni:SOIC-8" V 3575 4400 50  0001 C CNN
 F 3 "~" H 3300 4400 50  0001 C CNN
+F 4 "Y7471CT-ND" H 3300 4400 50  0001 C CNN "Digikey P/N"
 	1    3300 4400
 	0    -1   1    0
@@
 F 2 "LED_SMD:LED_0805_2012Metric" H 3800 4250 50  0001 C CNN
 F 3 "~" H 3800 4250 50  0001 C CNN
+F 4 "160-1423-1-ND" H 3800 4250 50  0001 C CNN "Digikey P/N"
 	1    3800 4250
 	-1   0    0    1
@@
 F 2 "LED_SMD:LED_0805_2012Metric" H 3800 4050 50  0001 C CNN
 F 3 "~" H 3800 4050 50  0001 C CNN
+F 4 "160-1423-1-ND" H 3800 4050 50  0001 C CNN "Digikey P/N"
 	1    3800 4050
 	-1   0    0    1
@@
 F 2 "LED_SMD:LED_0805_2012Metric" H 3800 4450 50  0001 C CNN
 F 3 "~" H 3800 4450 50  0001 C CNN
+F 4 "160-1423-1-ND" H 3800 4450 50  0001 C CNN "Digikey P/N"
 	1    3800 4450
 	-1   0    0    1
@@
 F 2 "LED_SMD:LED_0805_2012Metric" H 3800 4650 50  0001 C CNN
 F 3 "~" H 3800 4650 50  0001 C CNN
+F 4 "160-1423-1-ND" H 3800 4650 50  0001 C CNN "Digikey P/N"
 	1    3800 4650
 	-1   0    0    1

Commit message: update part numbers to 74ACT299
Parts:
- U6, U7, U8: value 74LS299 -> 74ACT299
Changed lines of the file:
@@
 P 6300 4000
 F 0 "U7" H 6450 4650 50  0000 C CNN
-F 1 "74LS299" H 6500 3250 50  0000 C CNN
+F 1 "74ACT299" H 6500 3250 50  0000 C CNN
 F 2 "Package_SO:SOIC-20W_7.5x12.8mm_P1.27mm" H 6300 4000 50  0001 C CNN
 F 3 "http://www.ti.com/lit/gpn/sn74LS299" H 6300 4000 50  0001 C CNN
@@
 P 6300 5950
 F 0 "U8" H 6450 6600 50  0000 C CNN
-F 1 "74LS299" H 6500 5200 50  0000 C CNN
+F 1 "74ACT299" H 6500 5200 50  0000 C CNN
 F 2 "Package_SO:SOIC-20W_7.5x12.8mm_P1.27mm" H 6300 5950 50  0001 C CNN
 F 3 "http://www.ti.com/lit/gpn/sn74LS299" H 6300 5950 50  0001 C CNN
@@
 P 6300 2050
 F 0 "U6" H 6450 2700 50  0000 C CNN
-F 1 "74LS299" H 6500 1300 50  0000 C CNN
+F 1 "74ACT299" H 6500 1300 50  0000 C CNN
 F 2 "Package_SO:SOIC-20W_7.5x12.8mm_P1.27mm" H 6300 2050 50  0001 C CNN
 F 3 "http://www.ti.com/lit/gpn/sn74LS299" H 6300 2050 50  0001 C CNN
